Commit message: change phoxi frame name and remove second phoxi

File: ur_e_description/urdf/ur5e_robot.urdf.xacro (robot description, xacro)
@@ -36,10 +36,10 @@
   <joint name="phoxi_osaka_frame_joint" type="fixed">
     <parent link="base_link" />
-    <child link = "phoxi_osaka_frame_link" />
+    <child link = "PhoXi3Dscanner_sensor" />
     <!--origin xyz="0 0 0" rpy="0 0 0" /-->
     <!--origin xyz="0.492 -0.101 0.957" rpy="2.991102168713803 0.019032241296778604 -1.586274049895831" /-->
     <origin xyz="0.492 -0.101 0.957" rpy="3.124909241602114 0.1507675271923597 1.5864488188586465" />
   </joint>
-  <link name="phoxi_osaka_frame_link">
+  <link name="PhoXi3Dscanner_sensor">
     <visual>
       <!--origin rpy="0 0 0" xyz="0 0 0"/-->
@@ -56,8 +56,8 @@
     </visual>
   </link>
-  <xacro:PhoXi3Dscanner scanner_parent = "base_link" scanner_name = "PhoXi3Dscanner" sensor_parent = "PhoXi3Dscanner" sensor_name = "PhoXi3Dscanner_sensor" >
-      <origin xyz="0 0 0" rpy="0 0 0" /> <!--PhoXi3Dscanner origin-->
-      <xacro:PhoXi3DscannerM_default_sensor_origin /> <!--Extrinsic calibration data-->
-      <xacro:PhoXi3DscannerM_meshes /> <!--meshes-->
-  </xacro:PhoXi3Dscanner>
+  <!--xacro:PhoXi3Dscanner scanner_parent = "base_link" scanner_name = "PhoXi3Dscanner" sensor_parent = "PhoXi3Dscanner" sensor_name = "PhoXi3Dscanner_sensor" -->
+      <!--origin xyz="0 0 0" rpy="0 0 0" /--> <!--PhoXi3Dscanner origin-->
+      <!--xacro:PhoXi3DscannerM_default_sensor_origin /--> <!--Extrinsic calibration data-->
+      <!--xacro:PhoXi3DscannerM_meshes /--> <!--meshes-->
+  <!--/xacro:PhoXi3Dscanner-->
 </robot>

Commit message: change package name from my_test_movit_script by pick_easy

File: ur_e_description/urdf/ur5e_robot.urdf.xacro (robot description, xacro)
@@ -27,5 +27,5 @@
       <origin rpy="0 0 0" xyz="0 0 0"/>
       <geometry>
-        <mesh filename="package://my_test_movit_script/ur5e_scene/robot_base.dae"/>
+        <mesh filename="package://pick_easy/ur5e_scene/robot_base.dae"/>
       </geometry>
     </visual>
@@ -49,5 +49,5 @@
       <geometry>
         <xacro:PhoXi3DscannerL_meshes />
-        <!--mesh filename="package://my_test_movit_script/ur5e_scene/robot_base.dae"/-->
+        <!--mesh filename="package://pick_easy/ur5e_scene/robot_base.dae"/-->
       </geometry>
       <material name="black">
